File: Radio_Kiosk_v2b/board.kicad_sch (KiCad schematic)
At the start: 188 parts, among them J1 USB-C PD in, J11 UART, J12 USB-C, J13 Lid LEDs, J2 DC in 18-26V, PJ-002BH 5.5x2.5, J3 Laptop out 15.6V, PJ-002BH 5.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, J5 RJ45 radio, J6 RJ45 laptop, J8 Fan 12V, J9 SWD, Q1 SI4470EY, Q10 2N7002, Q11 SI4470EY, Q13 SI4470EY, Q2 SI4470EY, Q20 AO4482, Q22 PSMN075-100MSEX, Q30 AO3400A, Q6 SI4470EY, Q7 SI4470EY, Q8 AOD4185, Q9 2N7002, SW1 RESET, SW2 BOOT0 (DFU), U1 LM74700-Q1, U10 TLV7011, U2 LM74700-Q1, U20 LM3478 54V boost, U21 TPS26600 eFuse, U22 LTC4279, U3 LMR33630 12V, U30 SN74AHCT1G125, U4 LMR33630 15.6V, U40 STM32F072CBT6, U41 INA180A1, U42 INA180A2, U43 LMV321, U5 LMR33630 5V, U50 CH224A, U51 AP2112K-3.3, U52 USBLC6-2SC6, U6 LM74700-Q1, U7 LM74700-Q1

Commit message: v2b: Filip's KiCad project (his routing, 2026-09-24 01:00) and the fixed copy: +3V3 net restored, SOIC-8 FET pins, net classes, GND stitching vias
Parts:
- removed Q1, Q11, Q13, Q2, Q6, Q7: SI4470EY, Package_SO:SOIC-8_3.9x4.9mm_P1.27mm, symbol Transistor_FET:Power_NMOS_60V
- added Q1, Q11, Q13, Q2, Q6, Q7: SI4470EY, Package_SO:SOIC-8_3.9x4.9mm_P1.27mm, symbol Transistor_FET:Power_NMOS_60V_SO8
- C141, C142, U51: LoonBlock 3f43bb1c-824e-4b38-b8a1-8f7f7ac2824c -> 47e99428-f54a-4653-af82-bd86ca40fa6a
- C143, J12, R122, R123, U52: LoonBlock e987e0ab-90c3-4600-95e2-bae4f6f81eca -> 51ad4a7d-c3ba-4aec-92c2-a387901ec1fe
Connections:
- net +12V: now also Q6.5 (D), Q6.6 (D), Q6.7 (D), Q6.8 (D)
- net +12V_BUCK: now also Q6.1 (S), Q6.2 (S), Q6.3 (S)
- net +15V6_S: now also Q7.1 (S), Q7.2 (S), Q7.3 (S)
- net +3V3: no longer BT4.2 (-), C110.2, C111.2, C112.2, C113.2, C114.2, C115.2, C116.2, C118.2, C130.2, C131.2, C132.2, C133.2, C134.2, C135.2, C136.2, C140.2, C141.2, C142.2, C143.2, C20.2, C21.2, C22.2, C23.2, C24.2, C25.2, C30.2, C31.2, C32.2, C34.2, C35.2, C36.2, C37.2, C40.2, C41.2, C42.2, C44.2, C45.2, C46.2, C47.2, C50.2, C51.2, C52.2, C54.2, C55.2, C56.2, C57.2, C60.2, C61.2, C62.2, C70.2, C90.2, C91.2, C97.2, C98.2, C99.2, D1.2 (A), D2.2 (A), D30.4 (VSS), D31.4 (VSS), D70.2 (A), J1.1 (SHELL), J1.2 (SHELL), J1.3 (SHELL), J1.4 (SHELL), J1.A1B12 (GND), J1.B1A12 (GND), J11.4 (Pin_4), J12.A1 (GND), J12.B1 (GND2), J12.S1 (SHIELD), J13.3 (GND), J2.2 (GND), J3.2 (GND), J9.4 (Pin_4), Q10.2 (S), Q9.2 (S), R100.2, R101.2, R104.2, R111.2, R120.2, R122.2, R123.2, R20.2, R21.2, R23.2, R31.2, R41.2, R51.2, R60.2, R61.2, R63.2, R72.2, R73.2, R74.2, R75.2, R76.2, R78.2, R83.2, R87.2, R89.2, R91.2, R92.2, R95.2, RT1.2, SW1.2, U1.2 (GND), U10.2 (VEE), U2.2 (GND), U20.4 (AGND), U20.5 (PGND), U21.17 (PAD), U21.3 (UVLO), U21.5 (OVP), U21.8 (RTN), U21.9 (GND), U22.10 (VEE), U22.4 (VSSK), U3.1 (PGND), U3.9 (AGND), U30.1 (OE), U30.3 (GND), U4.1 (PGND), U4.9 (AGND), U40.23 (VSS), U40.35 (VSS), U40.47 (VSS), U40.8 (VSSA), U41.2 (GND), U42.2 (GND), U43.2 (GND), U5.1 (PGND), U5.9 (AGND), U50.11 (EPAD), U51.2 (GND), U52.2 (GND), U6.2 (GND), U7.2 (GND)
- net BOOST_CS: now also Q20.1 (S), Q20.3 (S)
- net BOOST_DR: now also Q20.4 (G); no longer Q20.1 (G)
- net BOOST_SW: now also Q20.5 (D), Q20.6 (D), Q20.7 (D), Q20.8 (D), Q20.9 (D); no longer Q20.3 (D)
- net LAPTOP_OUT: now also Q7.5 (D), Q7.6 (D), Q7.7 (D), Q7.8 (D)
- net PASSIVE_EN: now also Q13.4 (G)
- net PORT_N: now also Q13.5 (D), Q13.6 (D), Q13.7 (D), Q13.8 (D)
- net TEST_LOAD: now also Q11.4 (G)
- net TEST_NODE: now also Q11.5 (D), Q11.6 (D), Q11.7 (D), Q11.8 (D)
- net U1_GATE: now also Q1.4 (G)
- net U2_GATE: now also Q2.4 (G)
- net U6_GATE: now also Q6.4 (G)
- net U7_GATE: now also Q7.4 (G)
- net VIN: now also Q1.5 (D), Q1.6 (D), Q1.7 (D), Q1.8 (D), Q2.5 (D), Q2.6 (D), Q2.7 (D), Q2.8 (D)
- net VIN_DC: now also Q2.1 (S), Q2.2 (S), Q2.3 (S)
- net VIN_USBS: now also Q1.1 (S), Q1.2 (S), Q1.3 (S)
- new net GND: BT4.2 (-), C110.2, C111.2, C112.2, C113.2, C114.2, C115.2, C116.2, C118.2, C130.2, C131.2, C132.2, C133.2, C134.2, C135.2, C136.2, C140.2, C141.2, C142.2, C143.2, C20.2, C21.2, C22.2, C23.2, C24.2, C25.2, C30.2, C31.2, C32.2, C34.2, C35.2, C36.2, C37.2, C40.2, C41.2, C42.2, C44.2, C45.2, C46.2, C47.2, C50.2, C51.2, C52.2, C54.2, C55.2, C56.2, C57.2, C60.2, C61.2, C62.2, C70.2, C90.2, C91.2, C97.2, C98.2, C99.2, D1.2 (A), D2.2 (A), D30.4 (VSS), D31.4 (VSS), D70.2 (A), J1.1 (SHELL), J1.2 (SHELL), J1.3 (SHELL), J1.4 (SHELL), J1.A1B12 (GND), J1.B1A12 (GND), J11.4 (Pin_4), J12.A1 (GND), J12.B1 (GND2), J12.S1 (SHIELD), J13.3 (GND), J2.2 (GND), J3.2 (GND), J9.4 (Pin_4), Q10.2 (S), Q11.1 (S), Q11.2 (S), Q11.3 (S), Q13.1 (S), Q13.2 (S), Q13.3 (S), Q9.2 (S), R100.2, R101.2, R104.2, R111.2, R120.2, R122.2, R123.2, R20.2, R21.2, R23.2, R31.2, R41.2, R51.2, R60.2, R61.2, R63.2, R72.2, R73.2, R74.2, R75.2, R76.2, R78.2, R83.2, R87.2, R89.2, R91.2, R92.2, R95.2, RT1.2, SW1.2, U1.2 (GND), U10.2 (VEE), U2.2 (GND), U20.4 (AGND), U20.5 (PGND), U21.17 (PAD), U21.3 (UVLO), U21.5 (OVP), U21.8 (RTN), U21.9 (GND), U22.10 (VEE), U22.4 (VSSK), U3.1 (PGND), U3.9 (AGND), U30.1 (OE), U30.3 (GND), U4.1 (PGND), U4.9 (AGND), U40.23 (VSS), U40.35 (VSS), U40.47 (VSS), U40.8 (VSSA), U41.2 (GND), U42.2 (GND), U43.2 (GND), U5.1 (PGND), U5.9 (AGND), U50.11 (EPAD), U51.2 (GND), U52.2 (GND), U6.2 (GND), U7.2 (GND)
