File: Radio_Kiosk_v2b/board.kicad_sch (KiCad schematic)
At the start: 188 parts, among them J1 USB-C PD in, J11 UART, J12 USB-C, J13 Lid LEDs, J2 DC in 18-26V, PJ-002BH 5.5x2.5, J3 Laptop out 15.6V, PJ-002BH 5.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, J5 RJ45 radio, J6 RJ45 laptop, J8 Fan 12V, J9 SWD, Q1 SI4470EY, Q10 2N7002, Q11 SI4470EY, Q13 SI4470EY, Q2 SI4470EY, Q20 AO4482, Q22 PSMN075-100MSEX, Q30 AO3400A, Q6 SI4470EY, Q7 SI4470EY, Q8 AOD4185, Q9 2N7002, SW1 RESET, SW2 BOOT0 (DFU), U1 LM74700-Q1, U10 TLV7011, U2 LM74700-Q1, U20 LM3478 54V boost, U21 TPS26600 eFuse, U22 LTC4279, U3 LMR33630 12V, U30 SN74AHCT1G125, U4 LMR33630 15.6V, U40 STM32F072CBT6, U41 INA180A1, U42 INA180A2, U43 LMV321, U5 LMR33630 5V, U50 CH224A, U51 AP2112K-3.3, U52 USBLC6-2SC6, U6 LM74700-Q1, U7 LM74700-Q1

Commit message: v2b schematic: audit fixes, port switch, LM3150 laptop rail
See loon scripts/build-radio-kiosk.ts for the design notes. Net changes are
listed in NETS-CHANGED.md. PCB not yet updated from this schematic.

Co-Authored-By: Claude Fable 5.1 <noreply@anthropic.com>
Parts:
- removed Q11, Q13: SI4470EY, Package_SO:SOIC-8_3.9x4.9mm_P1.27mm, symbol Transistor_FET:Power_NMOS_60V_SO8
- removed U4: LMR33630 15.6V, Package_SO:SOIC-8-1EP_3.9x4.9mm_P1.27mm_EP2.29x3mm, symbol Regulator_Switching:LMR33630
- removed U42: INA180A2, Package_TO_SOT_SMD:SOT-23-5, symbol Amplifier_Current:INA180A2
- removed U43: LMV321, Package_TO_SOT_SMD:SOT-23-5, symbol Amplifier_Operational:LMV321
- added C119: 47n, Capacitor_SMD:C_0805_2012Metric, symbol Device:C
- added C12, C120, C13, C16: 100n, Capacitor_SMD:C_0805_2012Metric, symbol Device:C
- added C14, C15: 10n, Capacitor_SMD:C_0805_2012Metric, symbol Device:C
- added C26: 4.7u/100V, Capacitor_SMD:C_1210_3225Metric, symbol Device:C
- added C3, C5: 100n/50V, Capacitor_SMD:C_0805_2012Metric, symbol Device:C
- added C4: 47u/63V, Capacitor_SMD:CP_Elec_8x10.5, symbol Device:C_Polarized
- added C48: 68n, Capacitor_SMD:C_0805_2012Metric, symbol Device:C
- added C49: 220p C0G, Capacitor_SMD:C_0805_2012Metric, symbol Device:C
- added C8: 1u/50V, Capacitor_SMD:C_1206_3216Metric, symbol Device:C
- added D23: BZT52C12 zener, Diode_SMD:D_SOD-123, symbol Device:D
- added Q11: AO3400A, Package_TO_SOT_SMD:SOT-23, symbol Device:Q_NMOS_GSD
- added Q12: SI4470EY, Package_SO:SOIC-8_3.9x4.9mm_P1.27mm, symbol Transistor_FET:Power_NMOS_60V_SO8
- added Q13: AO4482, Package_SO:SOIC-8_3.9x4.9mm_P1.27mm, symbol Transistor_FET:Power_NMOS_100V
- added Q23: DMP10H400SE, LCSC:SOT-223_L6.5-W3.5-P2.30-LS7.0-BR, symbol Transistor_FET:Power_PMOS_100V_SOT223
- added Q24: BSS123, Package_TO_SOT_SMD:SOT-23, symbol Device:Q_NMOS_GSD
- added Q25: 2N7002, Package_TO_SOT_SMD:SOT-23, symbol Device:Q_NMOS_GSD
- added Q40, Q41: AOD4184A, Package_TO_SOT_SMD:TO-252-2, symbol Transistor_FET:Power_NMOS_40V_DPAK
- added R113: 220R, Resistor_SMD:R_0805_2012Metric, symbol Device:R
- added R27, R46, R47, R66: 10k, Resistor_SMD:R_0805_2012Metric, symbol Device:R
- added R28: 47k, Resistor_SMD:R_0805_2012Metric, symbol Device:R
- added R29, R5, R6: 100k, Resistor_SMD:R_0805_2012Metric, symbol Device:R
- added R44: 523k 1%, Resistor_SMD:R_0805_2012Metric, symbol Device:R
- added R45: 681R 1%, Resistor_SMD:R_0805_2012Metric, symbol Device:R
- added R64: 1M 1%, Resistor_SMD:R_0805_2012Metric, symbol Device:R
- added R65: 56k 1%, Resistor_SMD:R_0805_2012Metric, symbol Device:R
- added U12: LM74700-Q1, Package_TO_SOT_SMD:SOT-23-6, symbol Power_Management:LM74700
- added U31: SN74AHCT1G125, Package_TO_SOT_SMD:SOT-23-5, symbol Logic_LevelTranslator:SN74AHCT1G125
- added U4: LM3150 15.75V 4.5A, LCSC:HTSSOP-14_L5.0-W4.4-P0.65-LS6.4-BL-EP, symbol Regulator_Controller:LM3150
- added U42: INA180A1, Package_TO_SOT_SMD:SOT-23-5, symbol Amplifier_Current:INA180A1
- added U43: MCP6001T-I/OT, Package_TO_SOT_SMD:SOT-23-5, symbol Amplifier_Operational:MCP6001-OT
- C117: value 10n -> 4.7n
- C141, C142, U51: LoonBlock 47e99428-f54a-4653-af82-bd86ca40fa6a -> e82a561b-776d-4694-8b0b-cd20f654fb10
- C143, R122, R123, U52: LoonBlock 51ad4a7d-c3ba-4aec-92c2-a387901ec1fe -> 624b899f-2b36-48da-b1f4-31f841ab14f8
- C25: value 47u/63V -> 47u/100V; LCSC C970680 -> C46224
- C42: value 1u -> 4.7u/16V
- C43: value 100n -> 470n/16V
- C44: value 22u/25V -> 10u/50V
- D1: value SMAJ28A TVS -> SMAJ22A TVS; LCSC C148227 -> C118189
- J12: LCSC C5143397 -> C165948; LoonBlock 51ad4a7d-c3ba-4aec-92c2-a387901ec1fe -> 624b899f-2b36-48da-b1f4-31f841ab14f8
- L3: value SRP7028A-100M 10u 5A -> MDA1040-150M 15u 6A; footprint Inductor_SMD:L_Bourns_SRP7028A_7.3x6.6mm -> LCSC:IND-SMD_L10.0-W10.0-APS10A40M470; LCSC C2687402 -> C2847554
- L4: value SRP7028A-100M 10u 5A -> MDA1040-100M 10u 8A; footprint Inductor_SMD:L_Bourns_SRP7028A_7.3x6.6mm -> LCSC:IND-SMD_L10.0-W10.0-APS10A40M470; LCSC C2687402 -> C2847553
- L5: value SRP7028A-100M 10u 5A -> SRP7028A-100M 10u 3.5A
- Q20: footprint Package_SO:SOIC-8-1EP_3.9x4.9mm_P1.27mm_EP2.41x3.3mm -> Package_SO:SOIC-8_3.9x4.9mm_P1.27mm
- R112: value 10R -> 0R
- R20: value 20m 1W -> 15m 1W
- R26, R63: value 100k -> 10k
- R40: value 100k -> 4.99k 1%
- R41: value 6.81k -> 126k 1%
- R85, R88: value 24R 1W -> 24R 2W pulse
- R86: value 100k -> 1M 1%
- R87: value 11.5k -> 115k 1%
Connections:
- net +12V: now also C50.1, C51.1, U21.3 (UVLO), U5.2 (VIN), U5.3 (EN)
- net +15V6_BUCK: now also R41.1, C49.1, U42.3 (IN+); no longer C44.1, R40.1
- net +15V6_S: now also C5.1, U42.4 (IN-)
- net +3V3: now also C120.1, U42.5 (VS), U43.5 (VDD)
- net +5V: now also C16.1, U31.5 (VCC)
- net BK_DRV: no longer Q10.3 (D)
- net BOOST_SW: no longer Q20.9 (D)
- net GND: now also D22.2 (A), R40.2, C119.2, C120.2, C13.2, C14.2, C15.2, C16.2, C26.2, C3.2, C4.2, C48.2, C5.2, C8.2, Q11.2 (S), Q13.1 (S), Q13.2 (S), Q13.3 (S), Q24.2 (S), Q25.2 (S), Q41.3 (S), R29.2, R6.2, R65.2, R66.2, U12.2 (GND), U31.1 (OE), U31.3 (GND), U4.14 (PGND), U4.15 (EP), U4.5 (SGND), U4.9 (SGND), U42.2 (GND), U43.2 (VSS); no longer Q9.2 (S), R41.2, U21.3 (UVLO)
- net LAPTOP_CC: now also U43.1 (OUT)
- net LAPTOP_EN: now also R46.1; no longer R92.1
- net LAPTOP_ILIM_N: now also U43.4 (IN-)
- net LAPTOP_ISENSE: now also R47.1, U42.1 (OUT)
- net LAPTOP_OUT: now also C8.1
- net LED_D0: no longer D30.1 (DIN), R103.2
- net LED_D2: now also R113.1; no longer J13.2 (DATA)
- net PACK_F: now also C12.2, Q12.1 (S), Q12.2 (S), Q12.3 (S), U12.3 (EN), U12.6 (ANODE); no longer Q8.3 (S), R80.1, R85.1, R86.1, R88.1
- net PACK_SENSE: now also C13.1
- net PASSIVE_EN: now also U31.2 (A)
- net PORT_N: now also Q13.5 (D), Q13.6 (D), Q13.7 (D), Q13.8 (D); no longer D22.2 (A)
- net PORT_P: now also D71.1 (K), Q23.2 (D), Q23.4 (D), R64.1; no longer C23.1, C24.1, C25.1, D20.1 (K), R22.1
- net PSE_AGND: no longer D71.1 (K)
- net TEST_LOAD: now also Q11.1 (G)
- net TEST_NODE: now also Q11.3 (D)
- net U4_FB: now also R40.1, R41.2, C49.2, U4.4 (FB); no longer R40.2, R41.1
- net U4_SW: now also Q40.3 (S), Q41.2 (D), R45.2, U4.10 (SW)
- net U4_VCC: now also U4.1 (VCC)
- net VIN: now also C44.1, C4.1, Q40.2 (D), R44.1, U4.2 (VIN); no longer C50.1, C51.1, U5.2 (VIN), U5.3 (EN)
- net VIN_DC: now also C3.1
- net VIN_SENSE: now also C14.1
- net VIN_USBS: now also R5.1; no longer U1.3 (EN)
- net PORT_SENSE: now reaches U40.18 (PB0/ADC8)
- net PORT_SENSE: now also C15.1, R64.2, R65.1
- net PORT_SW: now reaches U40.38 (PA15)
- net PORT_SW: now also Q24.1 (G), R29.1
- net USB_DIS: now reaches U40.46 (PB9)
- net USB_DIS: now also Q25.1 (G), R6.1
- net BK_KILL renamed BK_EN
- net U4_BOOT renamed U4_BST
- net U4_BST: now also U4.12 (BST)
- new net BK_ARM: Q10.3 (D), Q9.2 (S)
- new net BK_MID: Q12.5 (D), Q12.6 (D), Q12.7 (D), Q12.8 (D), Q8.3 (S), R80.1, R85.1, R86.1, R88.1, U12.4 (CATHODE)
- new net BOOST_OUT: C23.1, C24.1, C25.1, C26.1, D20.1 (K), D23.1 (K), Q23.3 (S), R22.1, R27.1
- new net LAPTOP_ISENSE_F: C119.1, R47.2, U43.3 (IN+)
- new net LED_D0R: D30.1 (DIN), R103.2
- new net LED_D2W: J13.2 (DATA), R113.2
- new net PASSIVE_EN5: Q13.4 (G), R66.1, U31.4 (Y)
- new net PORT_SW_D: Q24.3 (D), R28.2
- new net PORT_SW_G: D23.2 (A), Q23.1 (G), R27.2, R28.1
- new net U12_GATE: Q12.4 (G), U12.5 (GATE)
- new net U12_VCAP: C12.1, U12.1 (VCAP)
- new net U4_EN: R46.2, R92.1, U4.3 (EN)
- new net U4_HG: Q40.1 (G), U4.11 (HG)
- new net U4_ILIM: R45.1, U4.8 (ILIM)
- new net U4_LG: Q41.1 (G), U4.13 (LG)
- new net U4_RON: R44.2, U4.7 (RON)
- new net U4_SS: C48.1, U4.6 (SS)
- new net USB_EN: Q25.3 (D), R5.2, U1.3 (EN)
- no-connect marks 18 -> 17
Other:
- note added: "MCU: STM32F072CBT6 (128 KB), no radio. ADC: PA0 VIN_SENSE, PA1 PACK_SENSE (1M/115k), PA2 PASSIVE_IMON, PA3 TEMP_SENSE, PA4 FAN_SENSE, ADC5 USB_ISENSE (2 V = 5 A), ADC7 DCIN_SENSE, ADC8 PORT_SENSE (56 V = 2.97 V), ADC9 LAPTOP_ISENSE (0.4 V = 1 A). Out: PB2 LAPTOP_EN (off at reset), PA9 LAPTOP_ILIM_PWM (CC setpoint, 0.4 V = 1 A), PB12 TEST_LOAD, PB13 BOOST_SD (pulled up = off), PB14 PASSIVE_EN, PB1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"
- note added: "RADIO PORT: PORT_P = pins 4/5, PORT_N = pins 7/8 (Mode B). Unknown port: boost on, Q23 (PORT_SW) closed, PSE_EN: U22 probes the PD. Valid 802.3 signature within 700 ms: active, U22 powers PORT_N, 54 V on the port. No signature: PORT_SW open, PSE_EN off, PORT_P decays through R64, then PASSIVE_EN: U21 eFuse puts 12 V on PORT_P, Q13 grounds PORT_N. Never PORT_SW and PASSIVE_EN together. Empty port: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"
- note removed: "MCU: STM32F072CBT6 (128 KB), no radio. ADC: PA0 VIN_SENSE, PA1 PACK_SENSE, PA2 PASSIVE_IMON, PA3 TEMP_SENSE, PA4 FAN_SENSE. ADC5 USB_ISENSE (2 V = 5 A), ADC7 DCIN_SENSE, ADC9 LAPTOP_ISENSE (1 V = 1 A). Out: PB2 LAPTOP_EN (off at reset), PA9 LAPTOP_ILIM_PWM (CC setpoint, 1 V = 1 A), PB12 TEST_LOAD, PB13 BOOST_SD (pulled up = off), PB14 PASSIVE_EN, PB15 PSE_EN, PA6 FAN_PWM (TIM3_CH1), PA8 LED_DATA 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"
- note removed: "RADIO PORT: PORT_P = pins 4/5, PORT_N = pins 7/8 (Mode B). Active: +54V on PORT_P, the PSE switches PORT_N to ground. Passive: U21 eFuse puts 12 V on PORT_P, Q13 grounds PORT_N. Firmware never enables both: BOOST_SD high whenever PASSIVE_EN is high. Sequence: PSE detect first; valid signature = active; open/invalid = passive."

Commit message: v2b: E24 basic-library values and LCSC codes on every passive
Co-Authored-By: Claude Fable 5.1 <noreply@anthropic.com>
Parts:
- C1, C110, C111, C112, C114, C115, C116, C12, C120, C13, C131, C132, C133, C136, C16, C2, C33, C53, C6, C7, C99: LCSC (none) -> C28233
- C113, C135, C14, C15, C60: LCSC (none) -> C1710
- C117: LCSC (none) -> C1744
- C118, C134, C32, C52: LCSC (none) -> C28323
- C119, C21: LCSC (none) -> C53134
- C130, C42: LCSC (none) -> C1779
- C140, C61, C8: LCSC (none) -> C1848
- C141: LCSC (none) -> C15849; LoonBlock e82a561b-776d-4694-8b0b-cd20f654fb10 -> b0734d1b-18a3-4018-8acb-085b45cc16ab
- C142: LCSC (none) -> C19702; LoonBlock e82a561b-776d-4694-8b0b-cd20f654fb10 -> b0734d1b-18a3-4018-8acb-085b45cc16ab
- C143: LCSC (none) -> C19702; LoonBlock 624b899f-2b36-48da-b1f4-31f841ab14f8 -> d11f856a-3cdd-4692-a704-f2599572c964
- C20: LCSC (none) -> C1790
- C25: footprint Capacitor_SMD:CP_Elec_8x10.5 -> Capacitor_SMD:CP_Elec_10x10.5; LCSC C46224 -> C970681
- C3, C5: LCSC (none) -> C49678
- C31, C41, C51: LCSC (none) -> C5378
- C43: LCSC (none) -> C13967
- C48: value 68n -> 100n; LCSC (none) -> C28233
- C49: value 220p C0G -> 220p; LCSC (none) -> C107145
- C62, C70: LCSC (none) -> C24365
- C71: LCSC (none) -> C72067
- C90, C91: value 22u/50V -> 10u/50V; LCSC (none) -> C53084452
- D1: LCSC C118189 -> C148220
- D23: LCSC C8100 -> C12747
- J12, U52: LoonBlock 624b899f-2b36-48da-b1f4-31f841ab14f8 -> d11f856a-3cdd-4692-a704-f2599572c964
- Q23: LCSC C110374 -> C156277
- Q24: LCSC C8523 -> C78755
- Q40, Q41: LCSC C88370 -> C99124
- R100, R101, R29, R5, R6, R80, R89, R92, R97: LCSC (none) -> C149504
- R103, R106, R74, R75, R76, R77: LCSC (none) -> C17408
- R104: LCSC (none) -> C25271
- R105, R107, R111, R121, R24, R26, R27, R46, R47, R61, R62, R63, R66, R78, R79, R82, R83, R99: LCSC (none) -> C17414
- R112: LCSC (none) -> C17477
- R113: LCSC (none) -> C17557
- R120: LCSC (none) -> C17436
- R122, R123: LCSC (none) -> C23186; LoonBlock 624b899f-2b36-48da-b1f4-31f841ab14f8 -> d11f856a-3cdd-4692-a704-f2599572c964
- R20: LCSC (none) -> C44883
- R21: value 40.2k -> 47k; LCSC (none) -> C17713
- R22: value 402k -> 510k; LCSC (none) -> C17724
- R23: value 9.53k -> 12k; LCSC (none) -> C17444
- R25, R81: LCSC (none) -> C17513
- R28: LCSC (none) -> C17713
- R30: value 100k -> 220k; LCSC (none) -> C17556
- R31: value 9.09k -> 20k; LCSC (none) -> C4328
- R40: value 4.99k 1% -> 2k; LCSC (none) -> C17604
- R41: value 126k 1% -> 51k; LCSC (none) -> C17737
- R44: value 523k 1% -> 510k; LCSC (none) -> C17724
- R45: value 681R 1% -> 680R; LCSC (none) -> C17798
- R50: value 100k -> 12k; LCSC (none) -> C17444
- R51: value 24.9k -> 3k; LCSC (none) -> C17661
- R60: value 8.06k -> 5.1k; LCSC (none) -> C27834
- R64, R84, R86: LCSC (none) -> C17514
- R65: value 56k 1% -> 51k; LCSC (none) -> C17737
- R70: LCSC (none) -> C17415
- R71: LCSC (none) -> C17540
- R73: value 3.32k 1% -> 3.3k; LCSC (none) -> C26010
- R85, R88: LCSC (none) -> C25476
- R87: value 115k 1% -> 150k; LCSC (none) -> C17470
- R90, R94: value 100k -> 33k; LCSC (none) -> C17633
- R91, R95: value 14.0k -> 4.7k; LCSC (none) -> C17673
- R93, R96: LCSC (none) -> C2885416
- R98: LCSC (none) -> C17673
- SW1, SW2: LCSC (none) -> C231329
- U4: LCSC C130103 -> C48112
- U43: LCSC C7377 -> C116490
- U51: LoonBlock e82a561b-776d-4694-8b0b-cd20f654fb10 -> b0734d1b-18a3-4018-8acb-085b45cc16ab
Other:
- note added: "MCU: STM32F072CBT6 (128 KB), no radio. ADC: PA0 VIN_SENSE, PA1 PACK_SENSE (1M/150k), PA2 PASSIVE_IMON, PA3 TEMP_SENSE, PA4 FAN_SENSE, ADC5 USB_ISENSE (2 V = 5 A), ADC7 DCIN_SENSE, ADC8 PORT_SENSE (1M/51k, 56 V = 2.72 V), ADC9 LAPTOP_ISENSE (0.4 V = 1 A). Out: PB2 LAPTOP_EN (off at reset), PA9 LAPTOP_ILIM_PWM (CC setpoint, 0.4 V = 1 A), PB12 TEST_LOAD, PB13 BOOST_SD (pulled up = off), PB14 PASSIVE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"
- note removed: "MCU: STM32F072CBT6 (128 KB), no radio. ADC: PA0 VIN_SENSE, PA1 PACK_SENSE (1M/115k), PA2 PASSIVE_IMON, PA3 TEMP_SENSE, PA4 FAN_SENSE, ADC5 USB_ISENSE (2 V = 5 A), ADC7 DCIN_SENSE, ADC8 PORT_SENSE (56 V = 2.97 V), ADC9 LAPTOP_ISENSE (0.4 V = 1 A). Out: PB2 LAPTOP_EN (off at reset), PA9 LAPTOP_ILIM_PWM (CC setpoint, 0.4 V = 1 A), PB12 TEST_LOAD, PB13 BOOST_SD (pulled up = off), PB14 PASSIVE_EN, PB1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"

Commit message: v2b: STM32 in-stock code, 1N4148W basic
Co-Authored-By: Claude Fable 5.1 <noreply@anthropic.com>
Parts:
- C141, C142, U51: LoonBlock b0734d1b-18a3-4018-8acb-085b45cc16ab -> 17e3ad1a-da15-4558-93a1-678dcfd6073b
- C143, J12, R122, R123, U52: LoonBlock d11f856a-3cdd-4692-a704-f2599572c964 -> 8fcdefb5-9a17-437c-bb97-c1b1e7490cab
- D21, D40: LCSC C2099 -> C81598
- U40: LCSC C2969805 -> C81720

Commit message: v2b: U12 EN from BK_EN
Co-Authored-By: Claude Fable 5.1 <noreply@anthropic.com>
Parts:
- C141, C142, U51: LoonBlock 17e3ad1a-da15-4558-93a1-678dcfd6073b -> 20e56da2-67ae-45ce-a642-f7b455962625
- C143, J12, R122, R123, U52: LoonBlock 8fcdefb5-9a17-437c-bb97-c1b1e7490cab -> c2009584-855f-44c0-8de4-064ee0eaa827
Connections:
- net BK_EN: now also U12.3 (EN)
- net PACK_F: no longer U12.3 (EN)

Commit message: v2b: second audit fixes
Laptop rail: RON 820k (~190 kHz, clears the 725 ns minimum off-time at 20 V),
L4 15 uH, output bank 22u ceramic + 220u/25V polymer (ESR window), CFF 2.2n,
RLIM 750R, LAPTOP_OK divider to PC13 for a shorted jack. Port: eFuse ILIM
5.6k (in the 5.36k-120k range), dV/dt 47n, boost FB 499k (53.7 V, inside the
LTC4279 window over tolerance), 100k bleeder on BOOST_OUT. Comments fixed.

Co-Authored-By: Claude Fable 5.1 <noreply@anthropic.com>
Parts:
- removed C46, C47: 22u/25V, Capacitor_SMD:C_1210_3225Metric, symbol Device:C
- added C46: 220u/25V polymer, Capacitor_SMD:CP_Elec_6.3x7.7, symbol Device:C_Polarized
- added R42: 100k, Resistor_SMD:R_0805_2012Metric, symbol Device:R
- added R48: 47k, Resistor_SMD:R_0805_2012Metric, symbol Device:R
- added R49: 10k, Resistor_SMD:R_0805_2012Metric, symbol Device:R
- C141, C142, U51: LoonBlock 20e56da2-67ae-45ce-a642-f7b455962625 -> a62328a9-5e40-4b58-9a43-bf6b00971107
- C143, J12, R122, R123, U52: LoonBlock c2009584-855f-44c0-8de4-064ee0eaa827 -> 2ef44336-45cf-44b1-a4f5-5bb7dc2c018e
- C49: value 220p -> 2.2n; LCSC C107145 -> C28260
- C60: value 10n -> 47n; LCSC C1710 -> C53134
- L20: value MDA1365-330M 33u 4.5A -> MDA1365-330M 33u 9A
- L4: value MDA1040-100M 10u 8A -> MDA1040-150M 15u 6A; LCSC C2847553 -> C2847554
- R22: value 510k -> 499k 1%; LCSC C17724 -> C17721
- R44: value 510k -> 820k; LCSC C17724 -> C50136
- R45: value 680R -> 750R; LCSC C17798 -> C17818
- R60: value 5.1k -> 5.6k; LCSC C27834 -> C4382
Connections:
- net +15V6_BUCK: now also C46.1
- net BOOST_OUT: now also R42.1
- net GND: now also C46.2, R42.2, R49.2
- net LAPTOP_OUT: now also R48.1
- net LAPTOP_OK: now reaches U40.2 (PC13)
- net LAPTOP_OK: now also R48.2, R49.1

Commit message: v2b: interlocked laptop bypass for a 16 V brick
Q44 SI4401DDY from VIN to +15V6_S (source on VIN, body diode blocks), gate
through 10k/47k from Q45, BZT52C12 clamp. U45 TLV7011 compares VIN_SENSE with
a 2.2 V reference that only exists while PC14 LAPTOP_BYP is high, so the
bypass closes only below ~17.6 V and only on firmware's say-so. Parts along
the left edge by the laptop rail; front side only. tools: text-based clone
and placer; the pcbnew swap path dropped 44 footprints once and is retired.

Co-Authored-By: Claude Fable 5.1 <noreply@anthropic.com>
Parts:
- added C17: 100n, Capacitor_SMD:C_0805_2012Metric, symbol Device:C
- added D24: BZT52C12 zener, Diode_SMD:D_SOD-123, symbol Device:D
- added Q44: SI4401DDY, Package_SO:SOIC-8_3.9x4.9mm_P1.27mm, symbol Transistor_FET:Power_PMOS_40V_SO8
- added Q45: 2N7002, Package_TO_SOT_SMD:SOT-23, symbol Device:Q_NMOS_GSD
- added R10: 20k, Resistor_SMD:R_0805_2012Metric, symbol Device:R
- added R7, R9: 10k, Resistor_SMD:R_0805_2012Metric, symbol Device:R
- added R8: 47k, Resistor_SMD:R_0805_2012Metric, symbol Device:R
- added U45: TLV7011, Package_TO_SOT_SMD:SOT-23-5, symbol Comparator:TLV7011
- C141, C142, U51: LoonBlock a62328a9-5e40-4b58-9a43-bf6b00971107 -> 44e6b361-2241-4bbe-a4cb-adb02c11d269
- C143, J12, R122, R123, U52: LoonBlock 2ef44336-45cf-44b1-a4f5-5bb7dc2c018e -> bdb6fe49-29ef-497a-86d8-4a240e4bd89f
Connections:
- net +15V6_S: now also Q44.5 (D), Q44.6 (D), Q44.7 (D), Q44.8 (D)
- net +3V3: now also C17.1, U45.5 (VCC)
- net GND: now also C17.2, Q45.2 (S), R10.2, U45.2 (VEE)
- net VIN: now also D24.1 (K), Q44.1 (S), Q44.2 (S), Q44.3 (S), R7.1
- net VIN_SENSE: now also U45.4 (IN-)
- net LAPTOP_BYP: now reaches U40.3 (PC14/OSC32_IN)
- net LAPTOP_BYP: now also R9.1
- new net BYP_D: Q45.3 (D), R8.2
- new net BYP_EN: Q45.1 (G), U45.1 (OUT)
- new net BYP_G: D24.2 (A), Q44.4 (G), R7.2, R8.1
- new net BYP_REF: R10.1, R9.2, U45.3 (IN+)
