File: Radio_Kiosk_v2b/board.kicad_pcb (KiCad board)
At the start: 2 copper layers, 84 x 133 mm, 228 parts, among them J1 USB-C PD in, J11 UART, J12 USB-C, J13 Lid LEDs, J2 DC in 18-26V, PJ-002BH 5.5x2.5, J3 Laptop out 15.6V, PJ-002BH 5.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, J5 RJ45 radio, J6 RJ45 laptop, J8 Fan 12V, J9 SWD, Q1 SI4470EY, Q10 2N7002, Q11 AO3400A, Q12 SI4470EY, Q13 AO4482, Q2 SI4470EY, Q20 AO4482, Q22 PSMN075-100MSEX, Q23 DMP10H400SE, Q24 BSS123, Q25 2N7002, Q30 AO3400A, Q40 AOD4184A, Q41 AOD4184A, Q6 SI4470EY, Q7 SI4470EY, Q8 AOD4185, Q9 2N7002, SW1 RESET, SW2 BOOT0 (DFU), U1 LM74700-Q1, U10 TLV7011, U12 LM74700-Q1, U2 LM74700-Q1, U20 LM3478 54V boost, U21 TPS26600 eFuse, U22 LTC4279, U3 LMR33630 12V, U30 SN74AHCT1G125, U31 SN74AHCT1G125, U4 LM3150 15.75V 4.5A, U40 STM32F072CBT6, U41 INA180A1, U42 INA180A1, U43 MCP6001T-I/OT, U5 LMR33630 5V, U50 CH224A, U51 AP2112K-3.3, U52 USBLC6-2SC6, U6 LM74700-Q1, U7 LM74700-Q1

Commit message: v2b: corrected LCSC codes for the new parts, C25 as the 10 mm 100 V can
Co-Authored-By: Claude Fable 5.1 <noreply@anthropic.com>
Parts:
- C25: footprint Capacitor_SMD:CP_Elec_8x10.5 -> Capacitor_SMD:CP_Elec_10x10.5
Changed lines of the file:
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@@
 			)
 		)
-		(property "LCSC" "C130103"
+		(property "LCSC" "C48112"
 			(at 0 0 270)
 			(layer "F.SilkS")
@@
 			)
 		)
-		(property "LCSC" "C88370"
+		(property "LCSC" "C99124"
 			(at 0 0 0)
 			(layer "F.SilkS")
@@
 			)
 		)
-		(property "LCSC" "C8523"
+		(property "LCSC" "C78755"
 			(at 0 0 0)
 			(layer "F.SilkS")
@@
 		)
 	)
-	(footprint "Capacitor_SMD:CP_Elec_8x10.5"
+	(footprint "Capacitor_SMD:CP_Elec_10x10.5"
 		(layer "F.Cu")
 		(at 68.15 104.85)
-		(descr "SMD capacitor, aluminum electrolytic, Vishay 0810, 8.0x10.5mm, http://www.vishay.com/docs/28395/150crz.pdf")
+		(descr "SMD capacitor, aluminum electrolytic, Vishay 1010, 10.0x10.5mm, http://www.vishay.com/docs/28395/150crz.pdf")
 		(tags "capacitor electrolytic")
 		(property "Reference" "C25"
-			(at 0 -5.3 0)
+			(at 0 -6.3 0)
 			(layer "F.SilkS")
 			(effects
@@
 		)
 		(property "Value" "47u/100V"
-			(at 0 5.3 0)
+			(at 0 6.3 0)
 			(layer "F.Fab")
 			(effects
@@
 			)
 		)
-		(property "LCSC" "C46224"
+		(property "LCSC" "C970681"
 			(at 0 0 0)
 			(layer "F.SilkS")
@@
 		(duplicate_pad_numbers_are_jumpers no)
 		(fp_line
-			(start -5.6 -2.51)
-			(end -4.6 -2.51)
+			(start -6.85 -2.76)
+			(end -5.6 -2.76)
 			(stroke
 				(width 0.12)
@@
 		)
 		(fp_line
-			(start -5.1 -3.01)
-			(end -5.1 -2.01)
+			(start -6.225 -3.385)
+			(end -6.225 -2.135)
 			(stroke
 				(width 0.12)
@@
 		)
 		(fp_line
-			(start -4.36 -3.295563)
-			(end -4.36 -1.51)
+			(start -5.36 -4.295563)
+			(end -5.36 -1.51)
 			(stroke
 				(width 0.12)
@@
 		)
 		(fp_line
-			(start -4.36 -3.295563)
-			(end -3.295563 -4.36)
+			(start -5.36 -4.295563)
+			(end -4.295563 -5.36)
 			(stroke
 				(width 0.12)
@@
 		)
 		(fp_line
-			(start -4.36 3.295563)
-			(end -4.36 1.51)
+			(start -5.36 4.295563)
+			(end -5.36 1.51)
 			(stroke
 				(width 0.12)
@@
 		)
 		(fp_line
-			(start -4.36 3.295563)
-			(end -3.295563 4.36)
+			(start -5.36 4.295563)
+			(end -4.295563 5.36)
 			(stroke
 				(width 0.12)
@@
 		)
 		(fp_line
-			(start -3.295563 -4.36)
-			(end 4.36 -4.36)
+			(start -4.295563 -5.36)
+			(end 5.36 -5.36)
 			(stroke
 				(width 0.12)
@@
 		)
 		(fp_line
-			(start -3.295563 4.36)
-			(end 4.36 4.36)
+			(start -4.295563 5.36)
+			(end 5.36 5.36)
 			(stroke
 				(width 0.12)
@@
 		)
 		(fp_line
-			(start 4.36 -4.36)
-			(end 4.36 -1.51)
+			(start 5.36 -5.36)
+			(end 5.36 -1.51)
 			(stroke
 				(width 0.12)
@@
 		)
 		(fp_line
-			(start 4.36 4.36)
-			(end 4.36 1.51)
+			(start 5.36 5.36)
+			(end 5.36 1.51)
 			(stroke
 				(width 0.12)
@@
 		)
 		(fp_line
-			(start -6.15 -1.5)
-			(end -6.15 1.5)
+			(start -6.65 -1.5)
+			(end -6.65 1.5)
 			(stroke
 				(width 0.05)
@@
 		)
 		(fp_line
-			(start -6.15 1.5)
-			(end -4.5 1.5)
+			(start -6.65 1.5)
+			(end -5.5 1.5)
 			(stroke
 				(width 0.05)
@@
 		)
 		(fp_line
-			(start -4.5 -3.35)
-			(end -4.5 -1.5)
+			(start -5.5 -4.35)
+			(end -5.5 -1.5)
 			(stroke
 				(width 0.05)
@@
 		)
 		(fp_line
-			(start -4.5 -3.35)
-			(end -3.35 -4.5)
+			(start -5.5 -4.35)
+			(end -4.35 -5.5)
 			(stroke
 				(width 0.05)
@@
 		)
 		(fp_line
-			(start -4.5 -1.5)
-			(end -6.15 -1.5)
+			(start -5.5 -1.5)
+			(end -6.65 -1.5)
 			(stroke
 				(width 0.05)
@@
 		)
 		(fp_line
-			(start -4.5 1.5)
-			(end -4.5 3.35)
+			(start -5.5 1.5)
+			(end -5.5 4.35)
 			(stroke
 				(width 0.05)
@@
 		)
 		(fp_line
-			(start -4.5 3.35)
-			(end -3.35 4.5)
+			(start -5.5 4.35)
+			(end -4.35 5.5)
 			(stroke
 				(width 0.05)
@@
 		)
 		(fp_line
-			(start -3.35 -4.5)
-			(end 4.5 -4.5)
+			(start -4.35 -5.5)
+			(end 5.5 -5.5)
 			(stroke
 				(width 0.05)
@@
 		)
 		(fp_line
-			(start -3.35 4.5)
-			(end 4.5 4.5)
+			(start -4.35 5.5)
+			(end 5.5 5.5)
 			(stroke
 				(width 0.05)
@@
 		)
 		(fp_line
-			(start 4.5 -4.5)
-			(end 4.5 -1.5)
+			(start 5.5 -5.5)
+			(end 5.5 -1.5)
 			(stroke
 				(width 0.05)
@@
 		)
 		(fp_line
-			(start 4.5 -1.5)
-			(end 6.15 -1.5)
+			(start 5.5 -1.5)
+			(end 6.65 -1.5)
 			(stroke
 				(width 0.05)
@@
 		)
 		(fp_line
-			(start 4.5 1.5)
-			(end 4.5 4.5)
+			(start 5.5 1.5)
+			(end 5.5 5.5)
 			(stroke
 				(width 0.05)
@@
 		)
 		(fp_line
-			(start 6.15 -1.5)
-			(end 6.15 1.5)
+			(start 6.65 -1.5)
+			(end 6.65 1.5)
 			(stroke
 				(width 0.05)
@@
 		)
 		(fp_line
-			(start 6.15 1.5)
-			(end 4.5 1.5)
+			(start 6.65 1.5)
+			(end 5.5 1.5)
 			(stroke
 				(width 0.05)
@@
 		)
 		(fp_line
-			(start -4.25 -3.25)
-			(end -4.25 3.25)
+			(start -5.25 -4.25)
+			(end -5.25 4.25)
 			(stroke
 				(width 0.1)
@@
 		)
 		(fp_line
-			(start -4.25 -3.25)
-			(end -3.25 -4.25)
+			(start -5.25 -4.25)
+			(end -4.25 -5.25)
 			(stroke
 				(width 0.1)
@@
 		)
 		(fp_line
-			(start -4.25 3.25)
-			(end -3.25 4.25)
+			(start -5.25 4.25)
+			(end -4.25 5.25)
 			(stroke
 				(width 0.1)
@@
 		)
 		(fp_line
-			(start -3.562278 -1.5)
-			(end -2.762278 -1.5)
+			(start -4.558325 -1.7)
+			(end -3.558325 -1.7)
 			(stroke
 				(width 0.1)
@@
 		)
 		(fp_line
-			(start -3.25 -4.25)
-			(end 4.25 -4.25)
+			(start -4.25 -5.25)
+			(end 5.25 -5.25)
 			(stroke
 				(width 0.1)
@@
 		)
 		(fp_line
-			(start -3.25 4.25)
-			(end 4.25 4.25)
+			(start -4.25 5.25)
+			(end 5.25 5.25)
 			(stroke
 				(width 0.1)
@@
 		)
 		(fp_line
-			(start -3.162278 -1.9)
-			(end -3.162278 -1.1)
+			(start -4.058325 -2.2)
+			(end -4.058325 -1.2)
 			(stroke
 				(width 0.1)
@@
 		)
 		(fp_line
-			(start 4.25 -4.25)
-			(end 4.25 4.25)
+			(start 5.25 -5.25)
+			(end 5.25 5.25)
 			(stroke
 				(width 0.1)
@@
 		(fp_circle
 			(center 0 0)
-			(end 4 0)
+			(end 5 0)
 			(stroke
 				(width 0.1)
@@
 		)
 		(pad "1" smd roundrect
-			(at -3.7 0)
+			(at -4.2 0)
 			(size 4.4 2.5)
 			(layers "F.Cu" "F.Mask" "F.Paste")
@@
 		)
 		(pad "2" smd roundrect
-			(at 3.7 0)
+			(at 4.2 0)
 			(size 4.4 2.5)
 			(layers "F.Cu" "F.Mask" "F.Paste")
@@
 		)
 		(embedded_fonts no)
-		(model "${KICAD10_3DMODEL_DIR}/Capacitor_SMD.3dshapes/CP_Elec_8x10.5.step"
+		(model "${KICAD10_3DMODEL_DIR}/Capacitor_SMD.3dshapes/CP_Elec_10x10.5.step"
 			(offset
 				(xyz 0 0 0)
@@
 			)
 		)
-		(property "LCSC" "C88370"
+		(property "LCSC" "C99124"
 			(at 0 0 0)
 			(layer "F.SilkS")
@@
 			)
 		)
-		(property "LCSC" "C8100"
+		(property "LCSC" "C12747"
 			(at 0 0 90)
 			(layer "F.SilkS")
@@
 			)
 		)
-		(property "LCSC" "C110374"
+		(property "LCSC" "C156277"
 			(at 0 0 0)
 			(layer "F.SilkS")
@@
 			)
 		)
-		(property "LCSC" "C7377"
+		(property "LCSC" "C116490"
 			(at 0 0 0)
 			(layer "F.SilkS")
@@
 			)
 		)
-		(property "LCSC" "C118189"
+		(property "LCSC" "C148220"
 			(at 0 0 0)
 			(layer "F.SilkS")

Commit message: v2b: E24 basic-library values and LCSC codes on every passive
Co-Authored-By: Claude Fable 5.1 <noreply@anthropic.com>
Parts:
- C48: value 68n -> 100n
- C49: value 220p C0G -> 220p
- C90, C91: value 22u/50V -> 10u/50V
- R21: value 40.2k -> 47k
- R22: value 402k -> 510k
- R23: value 9.53k -> 12k
- R30: value 100k -> 220k
- R31: value 9.09k -> 20k
- R40: value 4.99k 1% -> 2k
- R41: value 126k 1% -> 51k
- R44: value 523k 1% -> 510k
- R45: value 681R 1% -> 680R
- R50: value 100k -> 12k
- R51: value 24.9k -> 3k
- R60: value 8.06k -> 5.1k
- R65: value 56k 1% -> 51k
- R73: value 3.32k 1% -> 3.3k
- R87: value 115k 1% -> 150k
- R90, R94: value 100k -> 33k
- R91, R95: value 14.0k -> 4.7k

Commit message: v2b: U12 EN from BK_EN
Co-Authored-By: Claude Fable 5.1 <noreply@anthropic.com>
Connections:
- U12 pad 3: PACK_F -> BK_EN
Changed lines of the file:
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@@
 			(layers "F.Cu" "F.Mask" "F.Paste")
 			(roundrect_rratio 0.25)
-			(net "PACK_F")
+			(net "BK_EN")
 		)
 		(pad "4" smd roundrect
