File: Radio_Kiosk_v2b/kicad/radio-kiosk-fixed.kicad_pcb (KiCad board)
At the start: 2 copper layers, 84 x 133 mm, 192 parts, among them J1 USB-C PD in, J11 UART, J12 Serial, J13 Lid LEDs, J2 DC in, J3 Laptop 15.6V, J5 RJ45 radio, J6 RJ45 laptop, J8 Fan 12V, J9 SWD, Q1 SI4470EY, Q10 2N7002, Q11 SI4470EY, Q13 SI4470EY, Q2 SI4470EY, Q20 AO4482, Q22 PSMN075-100MSEX, Q30 AO3400A, Q6 SI4470EY, Q7 SI4470EY, Q8 AOD4185, Q9 2N7002, SW1 RESET, SW2 BOOT0, U1 LM74700-Q1, U10 TLV7011, U2 LM74700-Q1, U20 LM3478 54V boost, U21 TPS26600 eFuse, U22 LTC4279, U3 LMR33630 12V, U30 SN74AHCT1G125, U4 LMR33630 15.6V, U40 STM32F072CBT6, U41 INA180A1, U42 INA180A2, U43 LMV321, U5 LMR33630 5V, U50 CH224A, U51 AP2112K-3.3, U52 USBLC6-2SC6, U6 LM74700-Q1, U7 LM74700-Q1

Commit message: v2b fixed board: FETs at 0 deg so the drains meet the hand routes; KiCad 10 DRC clean bar the receptacle's own pad gaps
Parts:
- turned Q1 to 0 degrees
- turned Q2 to 0 degrees
- turned Q7 to 0 degrees
Changed lines of the file:
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@@
 	(footprint "Package_SO:SOIC-8_3.9x4.9mm_P1.27mm"
 		(layer "F.Cu")
-		(at 75.87 57.48 180)
+		(at 75.87 57.48)
 		(descr "SOIC, 8 Pin (JEDEC MS-012AA, https://www.analog.com/media/en/package-pcb-resources/package/pkg_pdf/soic_narrow-r/r_8.pdf), generated with kicad-footprint-generator ipc_gullwing_generator.py")
 		(tags "SOIC SO")
@@
 	(footprint "Package_SO:SOIC-8_3.9x4.9mm_P1.27mm"
 		(layer "F.Cu")
-		(at 9.2 35.83 180)
+		(at 9.2 35.83)
 		(descr "SOIC, 8 Pin (JEDEC MS-012AA, https://www.analog.com/media/en/package-pcb-resources/package/pkg_pdf/soic_narrow-r/r_8.pdf), generated with kicad-footprint-generator ipc_gullwing_generator.py")
 		(tags "SOIC SO")
@@
 	(footprint "Package_SO:SOIC-8_3.9x4.9mm_P1.27mm"
 		(layer "F.Cu")
-		(at 72.81 44.38 180)
+		(at 72.81 44.38)
 		(descr "SOIC, 8 Pin (JEDEC MS-012AA, https://www.analog.com/media/en/package-pcb-resources/package/pkg_pdf/soic_narrow-r/r_8.pdf), generated with kicad-footprint-generator ipc_gullwing_generator.py")
 		(tags "SOIC SO")
@@
 		(start 77.24 10.8)
 		(end 75.3 10.8)
-		(width 0.6)
+		(width 0.3)
 		(layer "F.Cu")
 		(net "VIN_USB")
@@
 		(start 77.24 15.6)
 		(end 75.3 15.6)
-		(width 0.6)
+		(width 0.3)
 		(layer "F.Cu")
 		(net "VIN_USB")
