File: Radio_Kiosk_v2b/kicad/radio-kiosk-fixed.kicad_pcb (KiCad board)
At the start: 2 copper layers, 84 x 133 mm, 192 parts, among them J1 USB-C PD in, J11 UART, J12 Serial, J13 Lid LEDs, J2 DC in, J3 Laptop 15.6V, J5 RJ45 radio, J6 RJ45 laptop, J8 Fan 12V, J9 SWD, Q1 SI4470EY, Q10 2N7002, Q11 SI4470EY, Q13 SI4470EY, Q2 SI4470EY, Q20 AO4482, Q22 PSMN075-100MSEX, Q30 AO3400A, Q6 SI4470EY, Q7 SI4470EY, Q8 AOD4185, Q9 2N7002, SW1 RESET, SW2 BOOT0, U1 LM74700-Q1, U10 TLV7011, U2 LM74700-Q1, U20 LM3478 54V boost, U21 TPS26600 eFuse, U22 LTC4279, U3 LMR33630 12V, U30 SN74AHCT1G125, U4 LMR33630 15.6V, U40 STM32F072CBT6, U41 INA180A1, U42 INA180A2, U43 LMV321, U5 LMR33630 5V, U50 CH224A, U51 AP2112K-3.3, U52 USBLC6-2SC6, U6 LM74700-Q1, U7 LM74700-Q1

Commit message: v2b schematic: audit fixes, port switch, LM3150 laptop rail
See loon scripts/build-radio-kiosk.ts for the design notes. Net changes are
listed in NETS-CHANGED.md. PCB not yet updated from this schematic.

Co-Authored-By: Claude Fable 5.1 <noreply@anthropic.com>
Changed lines of the file:
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@@
 		(property "Value" "RJ45 laptop"
 			(at -9.3 -1.68 270)
-			(layer "F.Fab")
+			(layer "F.SilkS")
 			(effects
 				(font
@@
 		(property "Value" "RJ45 radio"
 			(at 0 -9.68 0)
-			(layer "F.Fab")
+			(layer "F.SilkS")
 			(effects
 				(font
@@
 		(property "Value" "USB-C PD in"
 			(at 5.7 -1.21 180)
-			(layer "F.Fab")
+			(layer "F.SilkS")
 			(effects
 				(font
@@
 		(property "Value" "DC in"
 			(at -5.2 2.5 90)
-			(layer "F.Fab")
+			(layer "F.SilkS")
 			(effects
 				(font
@@
 		(property "Value" "UART"
 			(at -2.5 7.62 180)
-			(layer "F.Fab")
+			(layer "F.SilkS")
 			(effects
 				(font
@@
 		(property "Value" "Serial"
 			(at -6.5 -4.15 270)
-			(layer "F.Fab")
+			(layer "F.SilkS")
 			(effects
 				(font
@@
 		(property "Value" "Fan 12V"
 			(at 0 -4.5 0)
-			(layer "F.Fab")
+			(layer "F.SilkS")
 			(effects
 				(font
@@
 		(property "Value" "SWD"
 			(at -2.5 7.81 180)
-			(layer "F.Fab")
+			(layer "F.SilkS")
 			(effects
 				(font
@@
 		(property "Value" "Laptop 15.6V"
 			(at 0.8 8 270)
-			(layer "F.Fab")
+			(layer "F.SilkS")
 			(effects
 				(font
@@
 		(property "Value" "Lid LEDs"
 			(at 0 3.5 0)
-			(layer "F.Fab")
+			(layer "F.SilkS")
 			(effects
 				(font
