File: Radio_Kiosk_v2d/board.kicad_sch (KiCad schematic)
At the start: 235 parts, among them J1 USB-C PD in, J11 UART, J12 USB-C, J13 Lid LEDs, J2 DC in 18-26V, PJ-002BH 5.5x2.5, J3 Laptop out 15.6V, PJ-002BH 5.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, J5 RJ45 radio, J6 RJ45 laptop, J8 Fan 12V, J9 SWD, Q1 SI4470EY, Q10 2N7002, Q11 AO3400A, Q12 SI4470EY, Q13 AO4482, Q2 SI4470EY, Q20 AO4482, Q22 PSMN075-100MSEX, Q23 DMP10H400SE, Q24 BSS123, Q25 2N7002, Q30 AO3400A, Q40 AOD4184A, Q41 AOD4184A, Q44 SI4401DDY, Q45 2N7002, Q6 SI4470EY, Q7 SI4470EY, Q8 AOD4185, Q9 2N7002, SW1 RESET, SW2 BOOT0 (DFU), U1 LM74700-Q1, U10 TLV7011, U12 LM74700-Q1, U2 LM74700-Q1, U20 LM3478 54V boost, U21 TPS26600 eFuse, U22 LTC4279, U3 LMR33630 12V, U30 SN74AHCT1G125, U31 SN74AHCT1G125, U4 LM3150 15.75V 4.5A, U40 STM32F072CBT6, U41 INA180A1, U42 INA180A1, U43 MCP6001T-I/OT, U45 TLV7011, U5 LMR33630 5V, U50 CH224A, U51 AP2112K-3.3, U52 USBLC6-2SC6, U6 LM74700-Q1, U7 LM74700-Q1

Commit message: v2d: fully routed, nothing foreign under the inductors, fab files
- Copper under L3/L4/L5/L20 ripped and re-routed with a keep-out: no signal on
  any layer, no foreign net on F.Cu or In2; power may pass on B.Cu under the
  In1 plane (FAN_N under L20 does).
- Last open net closed by a pin swap: USB_ISENSE PA0 -> PA3, PORT_SW PA3 ->
  PC15; schematic and firmware regenerated.
- KiCad DRC: 0 unconnected, no copper errors. fab/: gerbers, drill, JLC BOM
  and CPL.

Co-Authored-By: Claude Opus 5.5 <noreply@anthropic.com>
Parts:
- C141, C142, U51: LoonBlock 2f018ff6-2c0b-4b4b-956b-2965d561db95 -> 9137a5d2-afbc-4cba-83cd-3d5d258d1cc0
- C143, J12, R122, R123, U52: LoonBlock 02c0c3a3-9102-4f11-882e-52c10fdffd97 -> 0a62898d-dc2a-4fd0-afe6-f36c5335496a
Connections:
- net PORT_SW: now also U40.4 (PC15/OSC32_OUT); no longer U40.13 (PA3/ADC3)
- net USB_ISENSE: now also U40.13 (PA3/ADC3); no longer U40.10 (PA0/ADC0)

Commit message: v2d: C46 back to the 220u/25V polymer (C2981459), C44 to 10u/50V (C53084452)
A stale 'C44-C47 = 22u/25V 1210' line in the generator's LCSC table
overrode both: C46 became a 22u ceramic (the LM3150 needs the polymer's
ESR) and C44, on VIN up to 26 V, a 25 V part. Caught in JLC's matching sheet.

Co-Authored-By: Claude Opus 5.5 (1M context) <noreply@anthropic.com>
Parts:
- C44: LCSC C53084530 -> C53084452
- C46: LCSC C53084530 -> C2981459
Changed lines of the file:
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@@
 			)
 		)
-		(property "LCSC" "C53084530"
+		(property "LCSC" "C53084452"
 			(at 58.42 251.46 0)
 			(effects
@@
 			)
 		)
-		(property "LCSC" "C53084530"
+		(property "LCSC" "C2981459"
 			(at 165.10000000000002 251.46 0)
 			(effects
